File: Ram_chips_low.kicad_sch (KiCad schematic)
At the start: 10 parts, among them U25 MM5280, U26 MM5280, U27 MM5280, U28 MM5280, U40 MM5280, U41 MM5280, U42 MM5280, U43 MM5280, U6 74LS04, U7 74LS173

Commit message: Swap high and low RAM nibbles
Connections:
- net RAM_A0: now also U41.13 (A3)
- net RAM_A1: now also U41.15 (A5)
- net RAM_A10: now also U41.20 (A7)
- net RAM_A11: now also U41.21 (A8)
- net RAM_A2: now also U41.8 (A0)
- net RAM_A3: now also U41.10 (A2)
- net RAM_A4: now also U41.9 (A1)
- net RAM_A5: now also U41.14 (A4)
- net RAM_A6: now also U41.4 (A11)
- net RAM_A7: now also U41.19 (A6)
- net RAM_A8: now also U41.2 (A9)
- net RAM_A9: now also U41.3 (A10)
- net KIM_D0 renamed KIM_D4
- net KIM_D1 renamed KIM_D5
- net KIM_D2 renamed KIM_D6
- net KIM_D3 renamed KIM_D7
- net RAM_DOUT_0 renamed RAM_DOUT_4
- net RAM_DOUT_1 renamed RAM_DOUT_5
- net RAM_DOUT_2 renamed RAM_DOUT_6
- net RAM_DOUT_3 renamed RAM_DOUT_7
- net ~{DIN_0} renamed ~{DIN_4}
- net ~{DIN_1} renamed ~{DIN_5}
- net ~{DIN_2} renamed ~{DIN_6}
- net ~{DIN_3} renamed ~{DIN_7}
Changed lines of the file:
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@@
     (effects (font (size 1.27 1.27)) (justify left bottom))
   )
-  (label "~{DIN_2}" (at 56.642 205.232 180) (fields_autoplaced)
+  (label "~{DIN_6}" (at 56.642 205.232 180) (fields_autoplaced)
     (effects (font (size 1.27 1.27)) (justify right bottom))
   )
@@
     (effects (font (size 1.27 1.27)) (justify left bottom))
   )
-  (label "RAM_A8" (at 126.365 140.081 0) (fields_autoplaced)
+  (label "RAM_A8" (at 126.238 140.208 0) (fields_autoplaced)
     (effects (font (size 1.27 1.27)) (justify left bottom))
   )
@@
     (effects (font (size 1.27 1.27)) (justify left bottom))
   )
-  (label "~{DIN_1}" (at 56.642 215.392 180) (fields_autoplaced)
+  (label "~{DIN_5}" (at 56.642 215.392 180) (fields_autoplaced)
     (effects (font (size 1.27 1.27)) (justify right bottom))
   )
@@
     (effects (font (size 1.27 1.27)) (justify left bottom))
   )
-  (label "~{DIN_1}" (at 74.676 178.308 0) (fields_autoplaced)
+  (label "~{DIN_5}" (at 74.676 178.308 0) (fields_autoplaced)
     (effects (font (size 1.27 1.27)) (justify left bottom))
   )
@@
     (effects (font (size 1.27 1.27)) (justify left bottom))
   )
-  (label "RAM_A2" (at 126.365 162.941 0) (fields_autoplaced)
+  (label "RAM_A2" (at 126.238 163.068 0) (fields_autoplaced)
     (effects (font (size 1.27 1.27)) (justify left bottom))
   )
@@
     (effects (font (size 1.27 1.27)) (justify left bottom))
   )
-  (label "RAM_A5" (at 126.365 152.781 0) (fields_autoplaced)
+  (label "RAM_A5" (at 126.238 152.908 0) (fields_autoplaced)
     (effects (font (size 1.27 1.27)) (justify left bottom))
   )
@@
     (effects (font (size 1.27 1.27)) (justify left bottom))
   )
-  (label "RAM_A0" (at 126.365 155.321 0) (fields_autoplaced)
+  (label "RAM_A0" (at 126.238 155.448 0) (fields_autoplaced)
     (effects (font (size 1.27 1.27)) (justify left bottom))
   )
@@
     (effects (font (size 1.27 1.27)) (justify left bottom))
   )
-  (label "~{DIN_0}" (at 74.676 233.68 0) (fields_autoplaced)
+  (label "~{DIN_4}" (at 74.676 233.68 0) (fields_autoplaced)
     (effects (font (size 1.27 1.27)) (justify left bottom))
   )
@@
     (effects (font (size 1.27 1.27)) (justify left bottom))
   )
-  (label "~{DIN_3}" (at 138.176 67.564 0) (fields_autoplaced)
+  (label "~{DIN_7}" (at 138.176 67.564 0) (fields_autoplaced)
     (effects (font (size 1.27 1.27)) (justify left bottom))
   )
@@
     (effects (font (size 1.27 1.27)) (justify left bottom))
   )
-  (label "RAM_A3" (at 126.365 157.861 0) (fields_autoplaced)
+  (label "RAM_A3" (at 126.238 157.988 0) (fields_autoplaced)
     (effects (font (size 1.27 1.27)) (justify left bottom))
   )
@@
     (effects (font (size 1.27 1.27)) (justify left bottom))
   )
-  (label "~{DIN_1}" (at 138.176 178.308 0) (fields_autoplaced)
+  (label "~{DIN_5}" (at 138.176 178.308 0) (fields_autoplaced)
     (effects (font (size 1.27 1.27)) (justify left bottom))
   )
@@
     (effects (font (size 1.27 1.27)) (justify left bottom))
   )
-  (label "~{DIN_0}" (at 56.642 225.552 180) (fields_autoplaced)
+  (label "~{DIN_4}" (at 56.642 225.552 180) (fields_autoplaced)
     (effects (font (size 1.27 1.27)) (justify right bottom))
   )
@@
     (effects (font (size 1.27 1.27)) (justify left bottom))
   )
-  (label "~{DIN_3}" (at 56.642 195.072 180) (fields_autoplaced)
+  (label "~{DIN_7}" (at 56.642 195.072 180) (fields_autoplaced)
     (effects (font (size 1.27 1.27)) (justify right bottom))
   )
@@
     (effects (font (size 1.27 1.27)) (justify left bottom))
   )
-  (label "RAM_A7" (at 126.365 147.701 0) (fields_autoplaced)
+  (label "RAM_A7" (at 126.238 147.828 0) (fields_autoplaced)
     (effects (font (size 1.27 1.27)) (justify left bottom))
   )
@@
     (effects (font (size 1.27 1.27)) (justify left bottom))
   )
-  (label "~{DIN_2}" (at 74.676 122.936 0) (fields_autoplaced)
+  (label "~{DIN_6}" (at 74.676 122.936 0) (fields_autoplaced)
     (effects (font (size 1.27 1.27)) (justify left bottom))
   )
@@
     (effects (font (size 1.27 1.27)) (justify left bottom))
   )
-  (label "RAM_A1" (at 126.365 150.241 0) (fields_autoplaced)
+  (label "RAM_A1" (at 126.238 150.368 0) (fields_autoplaced)
     (effects (font (size 1.27 1.27)) (justify left bottom))
   )
@@
     (effects (font (size 1.27 1.27)) (justify left bottom))
   )
-  (label "RAM_A4" (at 126.365 160.401 0) (fields_autoplaced)
+  (label "RAM_A4" (at 126.238 160.528 0) (fields_autoplaced)
     (effects (font (size 1.27 1.27)) (justify left bottom))
   )
@@
     (effects (font (size 1.27 1.27)) (justify left bottom))
   )
-  (label "~{DIN_3}" (at 74.676 67.564 0) (fields_autoplaced)
+  (label "~{DIN_7}" (at 74.676 67.564 0) (fields_autoplaced)
     (effects (font (size 1.27 1.27)) (justify left bottom))
   )
@@
     (effects (font (size 1.27 1.27)) (justify left bottom))
   )
-  (label "~{DIN_0}" (at 138.176 233.68 0) (fields_autoplaced)
-    (effects (font (size 1.27 1.27)) (justify left bottom))
-  )
-  (label "RAM_A6" (at 126.365 135.001 0) (fields_autoplaced)
-    (effects (font (size 1.27 1.27)) (justify left bottom))
-  )
-  (label "RAM_A11" (at 126.365 142.621 0) (fields_autoplaced)
+  (label "~{DIN_4}" (at 138.176 233.68 0) (fields_autoplaced)
+    (effects (font (size 1.27 1.27)) (justify left bottom))
+  )
+  (label "RAM_A6" (at 126.238 135.128 0) (fields_autoplaced)
+    (effects (font (size 1.27 1.27)) (justify left bottom))
+  )
+  (label "RAM_A11" (at 126.238 142.748 0) (fields_autoplaced)
     (effects (font (size 1.27 1.27)) (justify left bottom))
   )
@@
     (effects (font (size 1.27 1.27)) (justify left bottom))
   )
-  (label "~{DIN_2}" (at 138.176 122.936 0) (fields_autoplaced)
-    (effects (font (size 1.27 1.27)) (justify left bottom))
-  )
-  (label "RAM_A9" (at 126.365 137.541 0) (fields_autoplaced)
+  (label "~{DIN_6}" (at 138.176 122.936 0) (fields_autoplaced)
+    (effects (font (size 1.27 1.27)) (justify left bottom))
+  )
+  (label "RAM_A9" (at 126.238 137.668 0) (fields_autoplaced)
     (effects (font (size 1.27 1.27)) (justify left bottom))
   )
@@
     (effects (font (size 1.27 1.27)) (justify left bottom))
   )
-  (label "RAM_A10" (at 126.365 145.161 0) (fields_autoplaced)
+  (label "RAM_A10" (at 126.238 145.288 0) (fields_autoplaced)
     (effects (font (size 1.27 1.27)) (justify left bottom))
   )
@@
     (effects (font (size 1.27 1.27)) (justify right))
   )
-  (hierarchical_label "KIM_D1" (shape input) (at 24.13 215.392 180) (fields_autoplaced)
-    (effects (font (size 1.27 1.27)) (justify right))
-  )
-  (hierarchical_label "RAM_DOUT_3" (shape output) (at 181.61 67.564 0) (fields_autoplaced)
+  (hierarchical_label "KIM_D5" (shape input) (at 24.13 215.392 180) (fields_autoplaced)
+    (effects (font (size 1.27 1.27)) (justify right))
+  )
+  (hierarchical_label "RAM_DOUT_7" (shape output) (at 181.61 67.564 0) (fields_autoplaced)
     (effects (font (size 1.27 1.27)) (justify left))
   )
-  (hierarchical_label "KIM_D3" (shape input) (at 24.13 195.072 180) (fields_autoplaced)
+  (hierarchical_label "KIM_D7" (shape input) (at 24.13 195.072 180) (fields_autoplaced)
     (effects (font (size 1.27 1.27)) (justify right))
   )
@@
     (effects (font (size 1.27 1.27)) (justify right))
   )
-  (hierarchical_label "KIM_D0" (shape input) (at 24.13 225.552 180) (fields_autoplaced)
-    (effects (font (size 1.27 1.27)) (justify right))
-  )
-  (hierarchical_label "RAM_DOUT_0" (shape output) (at 181.61 233.68 0) (fields_autoplaced)
+  (hierarchical_label "KIM_D4" (shape input) (at 24.13 225.552 180) (fields_autoplaced)
+    (effects (font (size 1.27 1.27)) (justify right))
+  )
+  (hierarchical_label "RAM_DOUT_4" (shape output) (at 181.61 233.68 0) (fields_autoplaced)
     (effects (font (size 1.27 1.27)) (justify left))
   )
@@
     (effects (font (size 1.27 1.27)) (justify right))
   )
-  (hierarchical_label "RAM_DOUT_2" (shape output) (at 181.61 122.936 0) (fields_autoplaced)
+  (hierarchical_label "RAM_DOUT_6" (shape output) (at 181.61 122.936 0) (fields_autoplaced)
     (effects (font (size 1.27 1.27)) (justify left))
   )
@@
     (effects (font (size 1.27 1.27)) (justify right))
   )
-  (hierarchical_label "KIM_D2" (shape input) (at 24.13 205.232 180) (fields_autoplaced)
-    (effects (font (size 1.27 1.27)) (justify right))
-  )
-  (hierarchical_label "RAM_DOUT_1" (shape output) (at 181.61 178.308 0) (fields_autoplaced)
+  (hierarchical_label "KIM_D6" (shape input) (at 24.13 205.232 180) (fields_autoplaced)
+    (effects (font (size 1.27 1.27)) (justify right))
+  )
+  (hierarchical_label "RAM_DOUT_5" (shape output) (at 181.61 178.308 0) (fields_autoplaced)
     (effects (font (size 1.27 1.27)) (justify left))
   )

Commit message: Routing completed
Connections:
- net RAM_DOUT_4: now also U27.16 (N/C), U42.16 (N/C)
- net RAM_DOUT_5: now also U26.16 (N/C), U41.16 (N/C)
- net RAM_DOUT_6: now also U28.16 (N/C), U43.16 (N/C)
- net RAM_DOUT_7: now also U25.16 (N/C), U40.16 (N/C)
Changed lines of the file:
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@@
   (junction (at 146.05 127.508) (diameter 0) (color 0 0 0 0)
   )
+  (junction (at 120.142 178.308) (diameter 0) (color 0 0 0 0)
+  )
+  (junction (at 117.856 122.936) (diameter 0) (color 0 0 0 0)
+  )
   (junction (at 120.142 185.166) (diameter 0) (color 0 0 0 0)
   )
+  (junction (at 122.428 233.68) (diameter 0) (color 0 0 0 0)
+  )
   (junction (at 81.534 115.316) (diameter 0) (color 0 0 0 0)
   )
@@
   (junction (at 33.274 195.072) (diameter 0) (color 0 0 0 0)
   )
+  (junction (at 115.57 67.564) (diameter 0) (color 0 0 0 0)
+  )
   (junction (at 83.312 117.856) (diameter 0) (color 0 0 0 0)
   )
@@
     (stroke (width 0) (type default))
   )
+  (wire (pts (xy 120.142 173.228) (xy 120.142 178.308))
+    (stroke (width 0) (type default))
+  )
   (wire (pts (xy 83.312 173.228) (xy 88.646 173.228))
     (stroke (width 0) (type default))
@@
     (stroke (width 0) (type default))
   )
+  (wire (pts (xy 177.038 173.228) (xy 177.038 178.308))
+    (stroke (width 0) (type default))
+  )
   (wire (pts (xy 126.238 82.296) (xy 150.622 82.296))
     (stroke (width 0) (type default))
   )
+  (wire (pts (xy 177.038 62.484) (xy 177.038 67.564))
+    (stroke (width 0) (type default))
+  )
   (bus (pts (xy 60.452 208.28) (xy 60.452 210.82))
     (stroke (width 0) (type default))
@@
     (stroke (width 0) (type default))
   )
+  (wire (pts (xy 176.022 173.228) (xy 177.038 173.228))
+    (stroke (width 0) (type default))
+  )
   (bus (pts (xy 60.452 77.216) (xy 60.452 79.756))
     (stroke (width 0) (type default))
@@
     (stroke (width 0) (type default))
   )
+  (wire (pts (xy 176.022 228.6) (xy 177.038 228.6))
+    (stroke (width 0) (type default))
+  )
   (bus (pts (xy 60.452 102.616) (xy 60.452 105.156))
     (stroke (width 0) (type default))
@@
     (stroke (width 0) (type default))
   )
+  (wire (pts (xy 114.046 228.6) (xy 122.428 228.6))
+    (stroke (width 0) (type default))
+  )
   (wire (pts (xy 62.992 195.58) (xy 88.646 195.58))
     (stroke (width 0) (type default))
@@
     (stroke (width 0) (type default))
   )
+  (wire (pts (xy 115.57 62.484) (xy 115.57 67.564))
+    (stroke (width 0) (type default))
+  )
   (bus (pts (xy 60.452 29.464) (xy 60.452 30.988))
     (stroke (width 0) (type default))
@@
     (stroke (width 0) (type default))
   )
+  (wire (pts (xy 176.022 62.484) (xy 177.038 62.484))
+    (stroke (width 0) (type default))
+  )
   (bus (pts (xy 123.698 203.2) (xy 123.698 205.74))
     (stroke (width 0) (type default))
@@
     (stroke (width 0) (type default))
   )
+  (wire (pts (xy 114.046 117.856) (xy 117.856 117.856))
+    (stroke (width 0) (type default))
+  )
   (wire (pts (xy 62.992 147.828) (xy 88.646 147.828))
     (stroke (width 0) (type default))
@@
     (stroke (width 0) (type default))
   )
+  (wire (pts (xy 177.038 228.6) (xy 177.038 233.68))
+    (stroke (width 0) (type default))
+  )
   (wire (pts (xy 88.646 115.316) (xy 81.534 115.316))
     (stroke (width 0) (type default))
@@
     (stroke (width 0) (type default))
   )
+  (wire (pts (xy 122.428 228.6) (xy 122.428 233.68))
+    (stroke (width 0) (type default))
+  )
   (wire (pts (xy 33.782 279.4) (xy 83.312 279.4))
     (stroke (width 0) (type default))
@@
     (stroke (width 0) (type default))
   )
+  (wire (pts (xy 176.022 117.856) (xy 177.038 117.856))
+    (stroke (width 0) (type default))
+  )
   (bus (pts (xy 60.452 36.068) (xy 60.452 37.084))
     (stroke (width 0) (type default))
@@
     (stroke (width 0) (type default))
   )
+  (wire (pts (xy 177.038 117.856) (xy 177.038 122.936))
+    (stroke (width 0) (type default))
+  )
   (wire (pts (xy 138.176 67.564) (xy 150.622 67.564))
     (stroke (width 0) (type default))
@@
     (stroke (width 0) (type default))
   )
+  (wire (pts (xy 117.856 117.856) (xy 117.856 122.936))
+    (stroke (width 0) (type default))
+  )
   (wire (pts (xy 126.238 137.668) (xy 150.622 137.668))
     (stroke (width 0) (type default))
@@
     (stroke (width 0) (type default))
   )
+  (wire (pts (xy 114.046 173.228) (xy 120.142 173.228))
+    (stroke (width 0) (type default))
+  )
   (bus (pts (xy 123.698 29.464) (xy 123.698 26.924))
     (stroke (width 0) (type default))
@@
     (stroke (width 0) (type default))
   )
+  (wire (pts (xy 114.046 62.484) (xy 115.57 62.484))
+    (stroke (width 0) (type default))
+  )
